Commit message: gpd cylinder works sometimes

File: deep_grasp_task/urdf/camera/camera.urdf.xacro (robot description, xacro)
@@ -4,6 +4,6 @@
   <xacro:include filename="$(find deep_grasp_task)/urdf/camera/camera_macro.urdf.xacro"/>
   <!-- camera side view for the cylinder -->
-  <xacro:kinect_camera parent_link="world" cam_py="-0.25" cam_pz="0.04"/>
+  <!-- <xacro:kinect_camera parent_link="world" cam_py="-0.25" cam_pz="0.04"/> -->
   <!-- overhead position -->
-  <!-- <xacro:kinect_camera parent_link="world" cam_px="0.5" cam_pz="0.7" cam_op="1.57079632679"/> -->
+  <xacro:kinect_camera parent_link="world" cam_px="0.5" cam_pz="0.7" cam_op="1.57079632679"/>
 </robot>

File: deep_grasp_task/urdf/objects/cylinder.urdf.xacro (robot description, xacro)
@@ -1,7 +1,7 @@
 <?xml version="1.0" encoding="utf-8"?>
 <robot xmlns:xacro="http://www.ros.org/wiki/xacro" name="cylinder">
-  <xacro:property name="r" value="0.02" />
-  <xacro:property name="h" value="0.25" />
-  <link name="cylinder_link">
+  <xacro:property name="r" value="0.015" />
+  <xacro:property name="h" value="0.15" />
+  <link name="object_link">
     <visual>
       <geometry>
@@ -24,5 +24,5 @@
     </collision>
   </link>
-  <gazebo reference="cylinder_link">
+  <gazebo reference="object_link">
     <!-- <material>Gazebo/Grey</material> -->
     <dampingFactor>0.005</dampingFactor>

File: deep_grasp_task/urdf/robots/panda_camera.urdf.xacro (robot description, xacro)
@@ -1,13 +1,13 @@
 <?xml version="1.0"?>
-<robot xmlns:xacro="http://www.ros.org/wiki/xacro" name="panda">
+<robot xmlns:xacro="http://www.ros.org/wiki/xacro" name="camera">
   <!-- Panda Arm + Hand -->
-  <xacro:include filename="$(find franka_description)/robots/panda_arm_hand.urdf.xacro"/>
+  <!-- <xacro:include filename="$(find franka_description)/robots/panda_arm_hand.urdf.xacro"/> -->
   <xacro:include filename="$(find deep_grasp_task)/urdf/camera/camera_macro.urdf.xacro"/>
   <!-- camera side view for the cylinder -->
-  <xacro:kinect_camera parent_link="panda_link0" cam_py="-0.25" cam_pz="0.04"/>
+  <xacro:kinect_camera parent_link="locobot_base_footprint" cam_py="-0.25" cam_pz="0.04"/>
   <!-- overhead position -->
   <!-- <xacro:kinect_camera parent_link="panda_link0" cam_px="0.5" cam_pz="0.7" cam_op="1.57079632679"/> -->
   <!-- Crank up the friction -->
-  <gazebo reference="panda_leftfinger">
+  <!-- <gazebo reference="panda_leftfinger">
     <mu1>100.0</mu1>
     <mu2>100.0</mu2>
@@ -16,4 +16,4 @@
     <mu1>100.0</mu1>
     <mu2>100.0</mu2>
-  </gazebo>
+  </gazebo> -->
 </robot>
