Commit message: gpd mustard works

File: deep_grasp_task/urdf/objects/barclamp.urdf.xacro (robot description, xacro)
@@ -13,6 +13,6 @@
     </collision>
 	<inertial>
-		<mass value="0.05"/>
-		<inertia ixx="0.1" iyy="0.1" izz="0.1" ixy="0.0" ixz="0.0" iyz="0.0"/>
+		<mass value="0.03"/>
+		<inertia ixx="0.05" iyy="0.05" izz="0.05" ixy="0.0" ixz="0.0" iyz="0.0"/>
 	</inertial>
   </link>
