Commit message: stack blocks working docker vnc

File: deep_grasp_task/urdf/objects/table.urdf.xacro (robot description, xacro)
@@ -1,32 +1,44 @@
+<?xml version="1.0"?>
 <robot name="table" xmlns:xacro="http://ros.org/wiki/xacro">
+  <xacro:arg name="x" default="0" />
+  <xacro:arg name="y" default="0" />
+  <xacro:arg name="z" default="0" />
+  <xacro:arg name="l" default="0.4" />
+  <xacro:arg name="h" default="0.0001" />
+  <xacro:arg name="w" default="0.5" />
   <link name="table">
     <inertial>
       <origin xyz="$(arg x) $(arg y) $(arg z)" />
-      <mass value="10.0" />
-      <inertia  ixx="1.0" ixy="0.0"  ixz="0.0"  iyy="100.0"  iyz="0.0"  izz="1.0" />
+      <mass value="1.0" />
+      <inertia ixx="1.0" ixy="0.0" ixz="0.0" iyy="1.0" iyz="0.0" izz="1.0" />
     </inertial>
     <visual>
-        <origin xyz="$(arg x) $(arg y) $(arg z)" />
+      <origin xyz="$(arg x) $(arg y) $(arg z)" />
       <geometry>
-          <box size="$(arg l) $(arg w) $(arg h)" />
+        <box size="$(arg l) $(arg w) $(arg h)" />
       </geometry>
     </visual>
     <collision>
-        <origin xyz="$(arg x) $(arg y) $(arg z)" />
+      <origin xyz="$(arg x) $(arg y) $(arg z)" />
       <geometry>
         <box size="$(arg l) $(arg w) $(arg h)" />
       </geometry>
     </collision>
-     <surface>
-        <friction>
-          <ode>
-            <mu>100</mu>
-            <mu2>100</mu2>
-          </ode>
-        </friction>
-      </surface>
+    <surface>
+      <friction>
+        <ode>
+          <mu>100</mu>
+          <mu2>100</mu2>
+        </ode>
+      </friction>
+    </surface>
   </link>
   <gazebo reference="table">
-    <material>Gazebo/Blue</material>
+    <visual>
+      <material>
+        <xacro:include filename="$(find deep_grasp_task)/urdf/colors.urdf.xacro" />
+        <xacro:color color="blue" />
+      </material>
+    </visual>
   </gazebo>
 </robot>
